File: aixa/aixa.kicad_pcb (KiCad board)
At the start: 2 copper layers, 61 x 57.5 mm, 6 parts, among them SW1 SW_SPDT

Commit message: mobile app
Routing:
- net /BCLK: track 0.00 -> 2.00 mm
Changed lines of the file:
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@@
 		(layer "Edge.Cuts")
+	)
+	(segment
+		(start 177 92)
+		(end 177 90)
+		(width 0.2)
+		(layer "F.Cu")
+		(net "/BCLK")
 	)
 	(zone
