File: aixa/aixa.kicad_sch (KiCad schematic)
At the start: 6 parts, among them SW1 SW_SPDT

Commit message: mobile app
Changed lines of the file:
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@@
 	)
 	(label "SCK"
-		(at 106.68 88.9 0)
+		(at 107.95 88.9 0)
 		(effects
 			(font
